Commit message: fix(lexus_description): fix xacro deprecated usage
Signed-off-by: Takayuki Murooka <takayuki5168@gmail.com>

File: lexus_description/urdf/vehicle.xacro (robot description, xacro)
@@ -2,5 +2,5 @@
 <robot xmlns:xacro="http://ros.org/wiki/xacro">
   <!-- load parameter -->
-  <xacro:property name="vehicle_info" value="${load_yaml('$(find lexus_description)/config/vehicle_info.param.yaml')}"/>
+  <xacro:property name="vehicle_info" value="${xacro.load_yaml('$(find lexus_description)/config/vehicle_info.param.yaml')}"/>
   <!-- vehicle body -->
   <link name="base_link">
